Commit message: Updated

File: skid/model/steer.xacro (robot description, xacro)
@@ -32,10 +32,7 @@
     </plugin>
   </gazebo>
-  <xacro:arg name="gpu" default="false"/>
-  <xacro:property name="gpu" value="$(arg gpu)" />
-  <xacro:arg name="organize_cloud" default="false"/>
-  <xacro:property name="organize_cloud" value="$(arg organize_cloud)" />
   <link name="link_chassis">
     <!-- pose and inertial -->
+    <pose>0 0 0.1 0 0 0</pose>
     <inertial>
       <mass value="5"/>
@@ -45,7 +42,7 @@
     </inertial>
     <!-- body -->
-    <collision>
+    <collision name="collision_chassis">
       <geometry>
-        <box size="0.38 0.38 0.08"/>
+        <box size="0.5 0.5 0.08"/>
       </geometry>
     </collision>
@@ -53,5 +50,5 @@
       <origin rpy="0 0 0" xyz="0 0 0"/>
       <geometry>
-        <box size="0.38 0.38 0.08"/>
+        <box size="0.5 0.5 0.08"/>
       </geometry>
       <material name="green"/>
@@ -66,8 +63,8 @@
         iyz="0" izz="0.025"/>
     </inertial>
-    <collision>
+    <collision name="link_front_right_wheel_collision">
       <origin rpy="0 1.5707 1.5707" xyz="0 0 0"/>
     <geometry>
-      <cylinder length="0.05" radius="0.05"/>
+      <cylinder length="0.05" radius="0.1"/>
     </geometry>
     </collision>
@@ -75,5 +72,5 @@
       <origin rpy="0 1.5707 1.5707" xyz="0 0 0"/>
     <geometry>
-      <cylinder length="0.05" radius="0.05"/>
+      <cylinder length="0.05" radius="0.1"/>
     </geometry>
     </visual>
@@ -86,8 +83,8 @@
         iyz="0" izz="0.025"/>
     </inertial>
-    <collision>
+    <collision name="link_front_left_wheel_collision">
       <origin rpy="0 1.5707 1.5707" xyz="0 0 0"/>
     <geometry>
-      <cylinder length="0.05" radius="0.05"/>
+      <cylinder length="0.05" radius="0.1"/>
     </geometry>
     </collision>
@@ -95,5 +92,5 @@
       <origin rpy="0 1.5707 1.5707" xyz="0 0 0"/>
     <geometry>
-      <cylinder length="0.05" radius="0.05"/>
+      <cylinder length="0.05" radius="0.1"/>
     </geometry>
     </visual>
@@ -106,8 +103,8 @@
         iyz="0" izz="0.025"/>
     </inertial>
-    <collision>
+    <collision name="link_back_right_wheel_collision">
       <origin rpy="0 1.5707 1.5707" xyz="0 0 0"/>
     <geometry>
-      <cylinder length="0.05" radius="0.05"/>
+      <cylinder length="0.05" radius="0.1"/>
     </geometry>
     </collision>
@@ -115,5 +112,5 @@
       <origin rpy="0 1.5707 1.5707" xyz="0 0 0"/>
     <geometry>
-      <cylinder length="0.05" radius="0.05"/>
+      <cylinder length="0.05" radius="0.1"/>
     </geometry>
     </visual>
@@ -126,8 +123,8 @@
         iyz="0" izz="0.025"/>
     </inertial>
-    <collision>
+    <collision name="link_back_left_wheel_collision">
       <origin rpy="0 1.5707 1.5707" xyz="0 0 0"/>
     <geometry>
-      <cylinder length="0.05" radius="0.05"/>
+      <cylinder length="0.05" radius="0.1"/>
     </geometry>
     </collision>
@@ -135,5 +132,5 @@
       <origin rpy="0 1.5707 1.5707" xyz="0 0 0"/>
     <geometry>
-      <cylinder length="0.05" radius="0.05"/>
+      <cylinder length="0.05" radius="0.1"/>
     </geometry>
     </visual>
@@ -141,54 +138,40 @@
   <!-- defining joints -->
   <joint name="front_right_wheel_joint" type="continuous">
-    <origin rpy="0 0 0" xyz="0.18 0.18 0"/>
+    <origin rpy="0 0 0" xyz="0.27 0.27 0"/>
     <child link="link_front_right_wheel"/>
     <parent link="link_chassis"/>
     <axis rpy="0 0 0" xyz="0 1 0"/>
     <limit effort="100" velocity="1"/>
+    <joint_properties damping="1.0" friction="1.0"/>
   </joint>
   <joint name="front_left_wheel_joint" type="continuous">
-    <origin rpy="0 0 0" xyz="0.18 -0.18 0"/>
+    <origin rpy="0 0 0" xyz="0.27 -0.27 0"/>
     <child link="link_front_left_wheel"/>
     <parent link="link_chassis"/>
     <axis rpy="0 0 0" xyz="0 1 0"/>
     <limit effort="100" velocity="1"/>
-    </joint>
+    <joint_properties damping="1.0" friction="1.0"/>
+  </joint>
   <joint name="back_right_wheel_joint" type="continuous">
-    <origin rpy="0 0 0" xyz="-0.20 0.18 0"/>
+    <origin rpy="0 0 0" xyz="-0.27 0.27 0"/>
     <child link="link_back_right_wheel"/>
     <parent link="link_chassis"/>
     <axis rpy="0 0 0" xyz="0 1 0"/>
     <limit effort="100" velocity="1"/>
+    <joint_properties damping="1.0" friction="1.0"/>
   </joint>
   <joint name="back_left_wheel_joint" type="continuous">
-    <origin rpy="0 0 0" xyz="-0.20 -0.18 0"/>
+    <origin rpy="0 0 0" xyz="-0.27 -0.27 0"/>
     <child link="link_back_left_wheel"/>
     <parent link="link_chassis"/>
     <axis rpy="0 0 0" xyz="0 1 0"/>
     <limit effort="100" velocity="1"/>
+    <joint_properties damping="1.0" friction="1.0"/>
   </joint>
-  <xacro:include filename="$(find velodyne_description)/urdf/HDL-32E.urdf.xacro"/>
-  <xacro:HDL-32E parent="link_chassis" name="velodyne2" topic="/velodyne_points2" organize_cloud="${organize_cloud}" hz="10" samples="220" gpu="${gpu}" min_angle="-1.57" max_angle="1.57">
-	  <origin xyz="0 0.1 0.075" rpy="0 0 0" />
-  </xacro:HDL-32E>
-  <gazebo reference="imu_link">
-    <gravity>true</gravity>
-    <sensor name="imu_sensor" type="imu">
-      <always_on>true</always_on>
-      <update_rate>100</update_rate>
-      <visualize>true</visualize>
-      <topic>__default_topic__</topic>
-      <plugin filename="libgazebo_ros_imu_sensor.so" name="imu_plugin">
-        <topicName>imu</topicName>
-        <bodyName>imu_link</bodyName>
-        <updateRateHZ>10.0</updateRateHZ>
-        <gaussianNoise>0.0</gaussianNoise>
-        <xyzOffset>0 0 0</xyzOffset>
-        <rpyOffset>0 0 0</rpyOffset>
-        <frameName>imu_link</frameName>
-        <initialOrientationAsReference>false</initialOrientationAsReference>
-      </plugin>
-      <pose>0 0 0 0 0 0</pose>
-    </sensor>
-  </gazebo>
+  <xacro:include filename="$(find skidsteer)/model/lidar.xacro"/>
+  <joint name="lidarGlue" type="fixed">
+    <origin rpy="0 0 0" xyz="0 0 0.05"/>
+    <parent link="link_chassis"/>
+    <child link="laz_base"/>
+  </joint>
 </robot>
