Commit message: wtf

File: skidsteer/model/steer.xacro (robot description, xacro)
@@ -32,7 +32,49 @@
     </plugin>
   </gazebo>
+  <xacro:arg name="gpu" default="false"/>
+  <xacro:property name="gpu" value="$(arg gpu)" />
+  <xacro:arg name="organize_cloud" default="false"/>
+  <xacro:property name="organize_cloud" value="$(arg organize_cloud)" />
+<!-- <gazebo> -->
+<!--   <sensor type="gpu_ray" name="HDL32E"> -->
+<!--     <visualize>true</visualize> -->
+<!--     <update_rate>10</update_rate> -->
+<!--     <ray> -->
+<!--       <scan> -->
+<!--         <horizontal> -->
+<!--           <samples>2187</samples> -->
+<!--           <resolution>1</resolution> -->
+<!--           <min_angle>3.14</min_angle> -->
+<!--           <max_angle>3.14</max_angle> -->
+<!--         </horizontal> -->
+<!--         <vertical> -->
+<!--           <samples>32</samples> -->
+<!--           <resolution>1</resolution> -->
+<!--           <min_angle>-${30.67*3.14/180.0}</min_angle> -->
+<!--           <max_angle> ${10.67*3.14/180.0}</max_angle> -->
+<!--         </vertical> -->
+<!--       </scan> -->
+<!--       <range> -->
+<!--         <min>0.3</min> -->
+<!--         <max>131</max> -->
+<!--         <resolution>0.001</resolution> -->
+<!--       </range> -->
+<!--       <noise> -->
+<!--         <type>gaussian</type> -->
+<!--         <mean>0.0</mean> -->
+<!--         <stddev>0.0</stddev> -->
+<!--       </noise> -->
+<!--     </ray> -->
+<!--     <plugin name="gazebo_ros_laser_controller" filename="libgazebo_ros_velodyne_gpu_laser.so"> -->
+<!--       <topicName>/velodyne_points</topicName> -->
+<!--       <frameName>laz_base</frameName> -->
+<!--       <organize_cloud>false</organize_cloud> -->
+<!--       <min_range>0.9</min_range> -->
+<!--       <max_range>130</max_range> -->
+<!--     </plugin> -->
+<!--   </sensor> -->
+<!-- </gazebo> -->
   <link name="link_chassis">
     <!-- pose and inertial -->
-    <pose>0 0 0.1 0 0 0</pose>
     <inertial>
       <mass value="5"/>
@@ -42,5 +84,5 @@
     </inertial>
     <!-- body -->
-    <collision name="collision_chassis">
+    <collision>
       <geometry>
         <box size="0.5 0.5 0.08"/>
@@ -63,5 +105,5 @@
         iyz="0" izz="0.025"/>
     </inertial>
-    <collision name="link_front_right_wheel_collision">
+    <collision>
       <origin rpy="0 1.5707 1.5707" xyz="0 0 0"/>
     <geometry>
@@ -83,5 +125,5 @@
         iyz="0" izz="0.025"/>
     </inertial>
-    <collision name="link_front_left_wheel_collision">
+    <collision>
       <origin rpy="0 1.5707 1.5707" xyz="0 0 0"/>
     <geometry>
@@ -103,5 +145,5 @@
         iyz="0" izz="0.025"/>
     </inertial>
-    <collision name="link_back_right_wheel_collision">
+    <collision>
       <origin rpy="0 1.5707 1.5707" xyz="0 0 0"/>
     <geometry>
@@ -123,5 +165,5 @@
         iyz="0" izz="0.025"/>
     </inertial>
-    <collision name="link_back_left_wheel_collision">
+    <collision>
       <origin rpy="0 1.5707 1.5707" xyz="0 0 0"/>
     <geometry>
@@ -143,5 +185,4 @@
     <axis rpy="0 0 0" xyz="0 1 0"/>
     <limit effort="100" velocity="1"/>
-    <joint_properties damping="1.0" friction="1.0"/>
   </joint>
   <joint name="front_left_wheel_joint" type="continuous">
@@ -151,5 +192,4 @@
     <axis rpy="0 0 0" xyz="0 1 0"/>
     <limit effort="100" velocity="1"/>
-    <joint_properties damping="1.0" friction="1.0"/>
   </joint>
   <joint name="back_right_wheel_joint" type="continuous">
@@ -159,5 +199,4 @@
     <axis rpy="0 0 0" xyz="0 1 0"/>
     <limit effort="100" velocity="1"/>
-    <joint_properties damping="1.0" friction="1.0"/>
   </joint>
   <joint name="back_left_wheel_joint" type="continuous">
@@ -167,11 +206,62 @@
     <axis rpy="0 0 0" xyz="0 1 0"/>
     <limit effort="100" velocity="1"/>
-    <joint_properties damping="1.0" friction="1.0"/>
-  </joint>
-  <xacro:include filename="$(find skidsteer)/model/lidar.xacro"/>
-  <joint name="lidarGlue" type="fixed">
-    <origin rpy="0 0 0" xyz="0 0 0.05"/>
-    <parent link="link_chassis"/>
-    <child link="laz_base"/>
-  </joint>
+  </joint>
+  <!-- <xacro:property name="base_radius" value="0.05"/> -->
+  <!-- <xacro:property name="base_height" value="0.05"/> -->
+  <!-- <xacro:property name="laz_radius" value="0.04"/> -->
+  <!-- <xacro:property name="laz_height" value="0.1"/> -->
+  <!--  -->
+  <!-- <link name="laz_base"> -->
+  <!--   <visual> -->
+  <!--     <geometry> -->
+  <!--       <cylinder length="${base_height}" radius="${base_radius}"/> -->
+  <!--     </geometry> -->
+  <!--   </visual> -->
+  <!--  -->
+  <!--   <collision> -->
+  <!--     <geometry> -->
+  <!--       <cylinder length="${base_height}" radius="${base_radius}"/> -->
+  <!--     </geometry> -->
+  <!--   </collision> -->
+  <!--  -->
+  <!--   <inertial> -->
+  <!--     <mass value="0.1"/> -->
+  <!--     <inertia ixx="${(1/12) * 0.1 * (3 * base_radius * base_radius + base_height * base_height)}" ixy="0" ixz="0" iyy="${(1/12) * 0.1 * (3 * base_radius * base_radius + base_height * base_height)}" iyz="0" izz="${(1/2) * 0.1 * base_radius * base_radius}"/> -->
+  <!--   </inertial> -->
+  <!-- </link> -->
+  <!--  -->
+  <!-- <link name="laz_rot"> -->
+  <!--   <visual> -->
+  <!--     <geometry> -->
+  <!--       <cylinder length="${laz_height}" radius="${laz_radius}"/> -->
+  <!--     </geometry> -->
+  <!--   </visual> -->
+  <!--  -->
+  <!--   <collision> -->
+  <!--     <geometry> -->
+  <!--       <cylinder length="${laz_height}" radius="${laz_radius}"/> -->
+  <!--     </geometry> -->
+  <!--   </collision> -->
+  <!--  -->
+  <!--   <inertial> -->
+  <!--     <mass value="0.1"/> -->
+  <!--     <inertia ixx="${(1/12) * 0.1 * (3 * laz_radius * laz_radius + laz_height * laz_height)}" ixy="0" ixz="0" iyy="${(1/12) * 0.1 * (3 * laz_radius * laz_radius + laz_height * laz_height)}" iyz="0" izz="${(1/2) * 0.1 * laz_radius * laz_radius}"/> -->
+  <!--   </inertial> -->
+  <!-- </link> -->
+  <!--  -->
+  <!-- <joint name="lazRot" type="continuous"> -->
+  <!--   <parent link="laz_base"/> -->
+  <!--   <child link="laz_rot"/> -->
+  <!--   <axis xyz="0 0 1"/> -->
+  <!--   <origin xyz = "0 0 ${base_height/2}"/> -->
+  <!-- </joint> -->
+  <!-- <joint name="lidarGlue" type="fixed"> -->
+  <!--   <origin rpy="0 0 0" xyz="0.1 0 0.05"/>      -->
+  <!--   <parent link="link_chassis"/> -->
+  <!--   <child link="laz_base"/> -->
+  <!-- </joint> -->
+  <xacro:include filename="$(find velodyne_description)/urdf/HDL-32E.urdf.xacro"/>
+  <xacro:HDL-32E parent="link_chassis" name="velodyne2" topic="/velodyne_points2" organize_cloud="${organize_cloud}" hz="10" samples="220" gpu="${gpu}">
+    <origin xyz="0 0.1 0.05" rpy="0 0 0" />
+  </xacro:HDL-32E>
 </robot>

Commit message: lol

File: skidsteer/model/steer.xacro (robot description, xacro)
@@ -169,6 +169,6 @@
   </joint>
   <xacro:include filename="$(find velodyne_description)/urdf/HDL-32E.urdf.xacro"/>
-  <xacro:HDL-32E parent="link_chassis" name="velodyne2" topic="/velodyne_points2" organize_cloud="${organize_cloud}" hz="10" samples="220" gpu="${gpu}" min_angle="-1.57" max_angle="1.57">
-	  <origin xyz="0 0.1 0.075" rpy="0 0 0" />
+  <xacro:HDL-32E parent="link_chassis" name="velodyne2" topic="/cloud_in" organize_cloud="${organize_cloud}" hz="10" samples="220" gpu="${gpu}" min_angle="-1.57" max_angle="1.57">
+    <origin xyz="0 0 0.05" rpy="0 0 0" />
   </xacro:HDL-32E>
   <gazebo reference="imu_link">
@@ -192,3 +192,2 @@
     </sensor>
   </gazebo>
-</robot>
