Commit message: lmao

File: depth/urdf/steer.xacro (robot description, xacro)
@@ -1,6 +1,6 @@
 <?xml version="1.0" ?>
 <robot name="skid_steer_bot" xmlns:xacro="http://www.ros.org/wiki/xacro">
-  <xacro:include filename="$(find gpskid)/urdf/materials.xacro"/>
-  <xacro:include filename="$(find gpskid)/urdf/steer.gazebo"/>
+  <xacro:include filename="$(find lidskid)/urdf/materials.xacro"/>
+  <xacro:include filename="$(find lidskid)/urdf/steer.gazebo"/>
   <link name="base_link"/>
   <joint name="base_joint" type="fixed">
@@ -57,6 +57,6 @@
     </visual>
     <inertial>
-      <mass value="1e-3"/>
-       <inertia ixx="1e-3" ixy="0" ixz="0" iyy="1e-3" iyz="0" izz="1e-3" />
+      <mass value="1"/>
+       <inertia ixx="1" ixy="0" ixz="0" iyy="1" iyz="0" izz="1" />
     </inertial>
   </link>
